File: Health_Watch/Health_Watch.kicad_sch (KiCad schematic)
At the start: 25 parts, among them J1 Conn_ARM_SWD_TagConnect_TC203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, J2 USB_C_Receptacle_PowerOnly_6P, J3 JST-PH-Conn, U1 STM32L476RGTx, U2 MCP73831-2-OT, X1 32KHz, X2 8MHz

Commit message: adding schematic and PCB layout
Parts:
- removed X2: 8MHz, symbol Device:Crystal
- added C10, C9: 4u7, Capacitor_SMD:C_0603_1608Metric, symbol Device:C
- added D1: D_Schottky, Diode_SMD:D_SOD-523, symbol Device:D_Schottky
- added D2: TVS Diode, Diode_SMD:D_SOD-923, symbol Diode:PTVS5V0Z1USK
- added FM1, FM2, FM3: Fiducial, Fiducial:Fiducial_0.75mm_Mask1.5mm, symbol Mechanical:Fiducial
- added J4: Conn_01x11, Connector_PinHeader_1.00mm:01x10_Conn_Hole, symbol Connector_Generic:Conn_01x11
- added R5, R6: 4k7, Resistor_SMD:R_0402_1005Metric, symbol Device:R
- added R7, R8: 10K, Resistor_SMD:R_0603_1608Metric, symbol Device:R
- added SW1: SW_Omron_B3FS, Button_Switch_THT:SW_TH_Tactile_Omron_B3F-10xx, symbol Switch:SW_Omron_B3FS
- added U2: MIC5365-3.3YD5, Package_TO_SOT_SMD:SOT-23-5, symbol Regulator_Linear:MIC5365-3.3YD5
- added X1: 8MHz, Crystal:Crystal_SMD_3225-4Pin_3.2x2.5mm, symbol Device:Crystal_GND24
- C1: renamed from C6; footprint (none) -> Capacitor_SMD:C_0603_1608Metric; Distrubutor Link (none) -> https://www.mouser.com/ProductDetail/TAIYO-YUDEN/LMK107BJ47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; Manufacturer (none) -> TAIYO YUDEN; Manufacturer Part Number (none) -> LMK107BJ475KA-T
- C11: footprint (none) -> Capacitor_SMD:C_0402_1005Metric; Distrubutor Link (none) -> https://www.mouser.com/ProductDetail/KYOCERA-AVX/0402X7R104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; Manufacturer (none) -> KYOCERA AVX; Manufacturer Part Number (none) -> 0402X7R104KT7AT
- C12: renamed from C9; footprint (none) -> Capacitor_SMD:C_0402_1005Metric; Distrubutor Link (none) -> https://www.mouser.com/ProductDetail/KEMET/C0402C200F5GACTU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; Manufacturer (none) -> KEMET; Manufacturer Part Number (none) -> C0402C200F5GACTU
- C13: renamed from C10; footprint (none) -> Capacitor_SMD:C_0402_1005Metric; Distrubutor Link (none) -> https://www.mouser.com/ProductDetail/KEMET/C0402C200F5GACTU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; Manufacturer (none) -> KEMET; Manufacturer Part Number (none) -> C0402C200F5GACTU
- C14: renamed from C7; footprint (none) -> Capacitor_SMD:C_0402_1005Metric; Distrubutor Link (none) -> https://www.mouser.com/ProductDetail/TAIYO-YUDEN/MBASU105SC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; Manufacturer (none) -> TAIYO YUDEN; Manufacturer Part Number (none) -> MBASU105SCH100JFNA01
- C15: renamed from C8; footprint (none) -> Capacitor_SMD:C_0402_1005Metric; Distrubutor Link (none) -> https://www.mouser.com/ProductDetail/TAIYO-YUDEN/MBASU105SC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; Manufacturer (none) -> TAIYO YUDEN; Manufacturer Part Number (none) -> MBASU105SCH100JFNA01
- C2: renamed from C1; footprint (none) -> Capacitor_SMD:C_0402_1005Metric; Distrubutor Link (none) -> https://www.mouser.com/ProductDetail/KYOCERA-AVX/0402X7R104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; Manufacturer (none) -> KYOCERA AVX; Manufacturer Part Number (none) -> 0402X7R104KT7AT
- C3: renamed from C2; footprint (none) -> Capacitor_SMD:C_0402_1005Metric; Distrubutor Link (none) -> https://www.mouser.com/ProductDetail/KYOCERA-AVX/0402X7R104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; Manufacturer (none) -> KYOCERA AVX; Manufacturer Part Number (none) -> 0402X7R104KT7AT
- C4: renamed from C3; footprint (none) -> Capacitor_SMD:C_0402_1005Metric; Distrubutor Link (none) -> https://www.mouser.com/ProductDetail/KYOCERA-AVX/0402X7R104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; Manufacturer (none) -> KYOCERA AVX; Manufacturer Part Number (none) -> 0402X7R104KT7AT
- C5: renamed from C4; footprint (none) -> Capacitor_SMD:C_0402_1005Metric; Distrubutor Link (none) -> https://www.mouser.com/ProductDetail/KYOCERA-AVX/0402X7R104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; Manufacturer (none) -> KYOCERA AVX; Manufacturer Part Number (none) -> 0402X7R104KT7AT
- C6: renamed from C5; footprint (none) -> Capacitor_SMD:C_0402_1005Metric; Distrubutor Link (none) -> https://www.mouser.com/ProductDetail/KYOCERA-AVX/0402X7R104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; Manufacturer (none) -> KYOCERA AVX; Manufacturer Part Number (none) -> 0402X7R104KT7AT
- C7: renamed from C13; footprint (none) -> Capacitor_SMD:C_0805_2012Metric; Distrubutor Link (none) -> https://www.mouser.com/ProductDetail/TAIYO-YUDEN/TMK212BBJ1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; Manufacturer (none) -> TAIYO YUDEN; Manufacturer Part Number (none) -> TMK212BBJ106KG8T
- C8: renamed from C12; footprint (none) -> Capacitor_SMD:C_0603_1608Metric; Distrubutor Link (none) -> https://www.mouser.com/ProductDetail/TAIYO-YUDEN/LMK107BJ47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; Manufacturer (none) -> TAIYO YUDEN; Manufacturer Part Number (none) -> LMK107BJ475KA-T
- J1: renamed from J3; footprint Connector_JST:JST_PH_S2B-PH-SM4-TB_1x02-1MP_P2.00mm_Horizontal -> Health_Watch:CONN_S2B-PH-K-S_JST; Distrubutor Link (none) -> https://www.digikey.com/en/products/detail/jst-sales-americ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; Manufacturer (none) -> JST Sales America Inc.; Manufacturer Part Number (none) -> S2B-PH-K-S
- J2: footprint (none) -> Connector_USB:USB_C_Receptacle_GCT_USB4125-xx-x_6P_TopMnt_Horizontal; Distrubutor Link (none) -> https://www.mouser.com/ProductDetail/GCT/USB4125-GF-A?qs=KU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; Manufacturer (none) -> GCT; Manufacturer Part Number (none) -> USB4125-GF-A
- R1: renamed from R5; footprint (none) -> Resistor_SMD:R_0402_1005Metric; Distrubutor Link (none) -> https://www.mouser.com/ProductDetail/Vishay-Beyschlag/MCS04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; Manufacturer (none) -> Vishay / Beyschlag; Manufacturer Part Number (none) -> MCS04020C5101FE000
- R2: renamed from R3; footprint (none) -> Resistor_SMD:R_0402_1005Metric; Distrubutor Link (none) -> https://www.mouser.com/ProductDetail/Vishay-Beyschlag/MCS04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; Manufacturer (none) -> Vishay / Beyschlag; Manufacturer Part Number (none) -> MCS04020C5101FE000
- R3: renamed from R4; footprint (none) -> Resistor_SMD:R_0402_1005Metric; Distrubutor Link (none) -> https://www.mouser.com/ProductDetail/Vishay-Beyschlag/MCS04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; Manufacturer (none) -> Vishay / Beyschlag; Manufacturer Part Number (none) -> MCS04020C5101FE000
- R4: renamed from R2; footprint (none) -> Resistor_SMD:R_0603_1608Metric; Distrubutor Link (none) -> https://www.mouser.com/ProductDetail/Vishay-Dale/CRCW060310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; Manufacturer (none) -> Vishay / Dale; Manufacturer Part Number (none) -> CRCW060310K0FKEA
- R9: renamed from R1; footprint (none) -> Resistor_SMD:R_0603_1608Metric; Distrubutor Link (none) -> https://www.mouser.com/ProductDetail/Panasonic/ERJ-PA3F3900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; Manufacturer (none) -> Panasonic; Manufacturer Part Number (none) -> ERJ-PA3F3900V
- U1: renamed from U2; Distrubutor Link (none) -> https://www.mouser.com/ProductDetail/Microchip-Technology/M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; Manufacturer (none) -> Microchip Technology; Manufacturer Part Number (none) -> MCP73831T-2ACI/OT
- U3: renamed from U1; Distrubutor Link (none) -> https://www.mouser.com/ProductDetail/STMicroelectronics/STM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; Manufacturer (none) -> STMicroelectronics; Manufacturer Part Number (none) -> STM32L476RGT6
- X2: renamed from X1; footprint (none) -> Crystal:Crystal_SMD_EuroQuartz_EQ161-2Pin_3.2x1.5mm; Distrubutor Link (none) -> https://www.mouser.com/ProductDetail/Epson-Timing/FC-135R-3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; Manufacturer (none) -> Epson Timing; Manufacturer Part Number (none) -> FC-135R 32.7680KA-A3
- renumbered J1 to J3
Connections:
- net +: now also J1.2 (Pin_2), C9.1, U2.1 (VIN), U2.3 (EN); no longer J1.1 (Pin_1)
- net +3V3: now also C10.1, J4.1 (Pin_1), R5.2, R6.2, R7.2, R8.2, U2.5 (VOUT)
- net GND: now also J1.1 (Pin_1), C10.2, C9.2, D2.2 (A), J4.11 (Pin_11), SW1.2, U2.2 (GND), X1.2, X1.4; no longer J1.2 (Pin_2)
- net HSE_IN: now also X1.3
- net SWD_NRST: now also J4.3 (Pin_3)
- net at C13.2, R9.1: now also X1.1
- net GPIO_PA2: now reaches U3.16 (PA2)
- net GPIO_PA2: now also J4.2 (Pin_2), R7.1, R8.1, SW1.1
- net TFT_DC: now reaches U3.17 (PA3)
- net TFT_DC: now also J4.4 (Pin_4)
- net SPI_SCK: now reaches U3.21 (PA5)
- net SPI_SCK: now also J4.5 (Pin_5)
- net SPI_MISO: now reaches U3.22 (PA6)
- net SPI_MISO: now also J4.6 (Pin_6)
- net SPI_MOSI: now reaches U3.23 (PA7)
- net SPI_MOSI: now also J4.7 (Pin_7)
- net TFT_TC: now reaches U3.26 (PB0)
- net TFT_TC: now also J4.8 (Pin_8)
- net I2C_SCL: now reaches U3.29 (PB10)
- net I2C_SCL: now also J4.9 (Pin_9), R6.1
- net I2C_SDA: now reaches U3.30 (PB11)
- net I2C_SDA: now also J4.10 (Pin_10), R5.1
- net +5V: now reaches C7.1, J2.A9 (VBUS), J2.B9 (VBUS)
- net +5V: now also D1.2 (A), D2.1 (K); no longer U1.4 (V_{DD})
- new net: D1.1 (K), U1.4 (V_{DD})
- no-connect marks 1 -> 36
Other:
- note added: "(off board)"
- note added: "Fiducial Markers \"
- note added: "Power Button"
- note added: "SPI and I2C Connection"
- note added: "USB-C Charging Li-Po Battery and +3V7 to +3V3 LDO Regulator"
- note removed: "USB-C Charging Li-Po Battery"
- moved on the sheet: C1, C13, C14, C15, C2, C3, C4, C5, C6, C7, C8, J1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
